File: Projects/Client Name/Project Name/Design/rev01/rev01_1/Example_Atik/Example_Atik.kicad_sch (KiCad schematic)
At the start: 0 parts

Commit message: update 2
designed schematic base and block diagram
Other:
- added sheet BLOCK DIAGRAM (BLOCK DIAGRAM.kicad_sch)
- added sheet CAN (CAN.kicad_sch)
- added sheet FILTERS (FILTERS.kicad_sch)
- added sheet MCU (MCU.kicad_sch)
- added sheet MECHANICAL (MECHANICAL.kicad_sch)
- added sheet MOSFET DRIVER (MOSFET DRIVER.kicad_sch)
- added sheet MOSFETs (MOSFETs.kicad_sch)
- added sheet OVERVIEW (OVERVIEW.kicad_sch)
- note added: "Atik_ESC_rev01_1"
- title: Example Project -> Atik_ESC_rev01_1
